File: kicad_protov2/sik_ledimössö.kicad_pcb (KiCad board)
At the start: 2 copper layers, 76 parts, among them J1 Conn_01x06_Pin, J2 Conn_01x02_Pin, U1 ATtiny861A-S

Commit message: Uusi leiska
Parts:
- D1, D10, D11, D12, D13, D14, D15, D16, D17, D18, D19, D2, D20, D21, D22, D23, D24, D25, D26, D27, D28, D29, D3, D30, D31, D32, D33, D34, D35, D36, D37, D38, D39, D4, D40, D41, D42, D43, D44, D45, D46, D47, D48, D49, D5, D50, D51, D52, D53, D54, D55, D56, D57, D58, D59, D6, D60, D61, D62, D63, D64, D7, D8, D9: footprint LED_THT:LED_D5.0mm -> Library_zani:LED_D5.0mm_mod
- R2, R3, U1: moved to F.Cu
- moved R4 101.4 mm to (128.5, 144.0), turned to -45 degrees
- moved R5 97.0 mm to (129.5, 134.6), turned to 0 degrees
- moved R6 96.6 mm to (115.8, 139.2)
- moved R7 84.3 mm to (103.6, 122.4), turned to 180 degrees
- moved R8 83.9 mm to (114.3, 112.8), turned to 90 degrees
- moved C1 79.9 mm to (100.6, 128.1), turned to -90 degrees
- moved R3 74.2 mm to (116.3, 137.2)
- moved R1 73.2 mm to (118.9, 112.8), turned to 90 degrees
- moved R2 66.9 mm to (111.7, 136.7)
- moved J2 65.4 mm to (104.6, 126.5), turned to 0 degrees
- moved J1 46.8 mm to (121.9, 127.1), turned to 180 degrees
- moved U1 44.1 mm to (112.2, 127.1)
- moved D52 13.9 mm to (88.4, 137.3), turned to 180 degrees
- moved D53 13.0 mm to (92.2, 132.1), turned to 180 degrees
- moved D54 11.7 mm to (96.0, 126.7), turned to 180 degrees
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Routing:
- net Net-(D1-K): track 0.00 -> 317.8 mm, vias 0 -> 7
- net Net-(D16-K): track 0.00 -> 314.8 mm, vias 0 -> 8
- net Net-(D10-K): track 0.00 -> 314.8 mm, vias 0 -> 6
- net Net-(D15-K): track 0.00 -> 307.9 mm, vias 0 -> 9
- net Net-(D13-K): track 0.00 -> 294.3 mm, vias 0 -> 7
- net Net-(D11-K): track 0.00 -> 275.0 mm, vias 0 -> 7
- net Net-(D14-K): track 0.00 -> 269.5 mm, vias 0 -> 6
- net Net-(D12-K): track 0.00 -> 237.0 mm, vias 0 -> 7
- net Net-(D25-A): track 0.00 -> 111.4 mm, vias 0 -> 1
- net Net-(D17-A): track 0.00 -> 93.2 mm, vias 0 -> 1
- net Net-(D41-A): track 0.00 -> 91.1 mm, vias 0 -> 3
- net Net-(D33-A): track 0.00 -> 87.2 mm
- net Net-(D10-A): track 0.00 -> 71.3 mm, vias 0 -> 1
- net Net-(D1-A): track 0.00 -> 64.9 mm
- net Net-(D49-A): track 0.00 -> 61.7 mm
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Other:
- board outline added: 96.5 x 161.3 mm
