File: kicad_selka_mk1/kicad_selka_mk1.kicad_pcb (KiCad board)
At the start: 2 copper layers, 103.1 x 218.5 mm, 103 parts, among them J1 Conn_01x06_Pin, J10 Conn_01x01_Pin, J11 Conn_01x01_Pin, J12 Conn_01x01_Pin, J13 Conn_01x01_Pin, J14 Conn_01x01_Pin, J15 Conn_01x01_Pin, J16 Conn_01x01_Pin, J17 Conn_01x01_Pin, J18 Conn_01x01_Pin, J19 Conn_01x01_Pin, J2 Conn_01x02_Pin, J20 Conn_01x01_Pin, J21 Conn_01x01_Pin, J22 Conn_01x01_Pin, J23 Conn_01x01_Pin, J24 Conn_01x01_Pin, J25 Conn_01x01_Pin, J26 Conn_01x01_Pin, J27 Conn_01x01_Pin, J28 Conn_01x01_Pin, J3 Conn_01x01_Pin, J4 Conn_01x01_Pin, J5 Conn_01x01_Pin, J6 Conn_01x01_Pin, J7 Conn_01x01_Pin, J8 Conn_01x01_Pin, J9 Conn_01x01_Pin, U1 ATtiny861A-S

Commit message: selkäsalama mk1 done
Parts:
- removed the J1 at (57.8, 95.2)
- added J28: Conn_01x01_Pin, TestPoint:TestPoint_Pad_1.0x1.0mm, B.Cu at (104.9, 127.6)
- added J29: Conn_01x01_Pin, TestPoint:TestPoint_Pad_1.0x1.0mm, B.Cu at (102.4, 132.0)
- added J30: Conn_01x01_Pin, TestPoint:TestPoint_Pad_1.0x1.0mm, B.Cu at (101.2, 128.5)
- added J31: Conn_01x01_Pin, TestPoint:TestPoint_Pad_1.0x1.0mm, B.Cu at (114.6, 115.2)
- J1: renamed from J3; footprint Connector_PinSocket_2.54mm:PinSocket_1x01_P2.54mm_Vertical -> Connector_Pin:Pin_D0.7mm_L6.5mm_W1.8mm_FlatFork
- J10: renamed from J12; footprint Connector_PinSocket_2.54mm:PinSocket_1x01_P2.54mm_Vertical -> Connector_Pin:Pin_D0.7mm_L6.5mm_W1.8mm_FlatFork
- J11: renamed from J13; footprint Connector_PinSocket_2.54mm:PinSocket_1x01_P2.54mm_Vertical -> Connector_Pin:Pin_D0.7mm_L6.5mm_W1.8mm_FlatFork
- J12: renamed from J14; footprint Connector_PinSocket_2.54mm:PinSocket_1x01_P2.54mm_Vertical -> Connector_Pin:Pin_D0.7mm_L6.5mm_W1.8mm_FlatFork
- J13: renamed from J15; footprint Connector_PinSocket_2.54mm:PinSocket_1x01_P2.54mm_Vertical -> Connector_Pin:Pin_D0.7mm_L6.5mm_W1.8mm_FlatFork
- J14: renamed from J16; footprint Connector_PinSocket_2.54mm:PinSocket_1x01_P2.54mm_Vertical -> Connector_Pin:Pin_D0.7mm_L6.5mm_W1.8mm_FlatFork
- J15: renamed from J17; footprint Connector_PinSocket_2.54mm:PinSocket_1x01_P2.54mm_Vertical -> Connector_Pin:Pin_D0.7mm_L6.5mm_W1.8mm_FlatFork
- J16: renamed from J18; footprint Connector_PinSocket_2.54mm:PinSocket_1x01_P2.54mm_Vertical -> Connector_Pin:Pin_D0.7mm_L6.5mm_W1.8mm_FlatFork
- J17: renamed from J19; footprint Connector_PinSocket_2.54mm:PinSocket_1x01_P2.54mm_Vertical -> Connector_Pin:Pin_D0.7mm_L6.5mm_W1.8mm_FlatFork
- J18: renamed from J20; footprint Connector_PinSocket_2.54mm:PinSocket_1x01_P2.54mm_Vertical -> Connector_Pin:Pin_D0.7mm_L6.5mm_W1.8mm_FlatFork
- J19: renamed from J21; footprint Connector_PinSocket_2.54mm:PinSocket_1x01_P2.54mm_Vertical -> Connector_Pin:Pin_D0.7mm_L6.5mm_W1.8mm_FlatFork
- J2: renamed from J4; footprint Connector_PinSocket_2.54mm:PinSocket_1x01_P2.54mm_Vertical -> Connector_Pin:Pin_D0.7mm_L6.5mm_W1.8mm_FlatFork
- J20: renamed from J22; footprint Connector_PinSocket_2.54mm:PinSocket_1x01_P2.54mm_Vertical -> Connector_Pin:Pin_D0.7mm_L6.5mm_W1.8mm_FlatFork
- J21: renamed from J23; footprint Connector_PinSocket_2.54mm:PinSocket_1x01_P2.54mm_Vertical -> Connector_Pin:Pin_D0.7mm_L6.5mm_W1.8mm_FlatFork
- J22: renamed from J24; footprint Connector_PinSocket_2.54mm:PinSocket_1x01_P2.54mm_Vertical -> Connector_Pin:Pin_D0.7mm_L6.5mm_W1.8mm_FlatFork
- J23: renamed from J25; footprint Connector_PinSocket_2.54mm:PinSocket_1x01_P2.54mm_Vertical -> Connector_Pin:Pin_D0.7mm_L6.5mm_W1.8mm_FlatFork
- J24: renamed from J26; footprint Connector_PinSocket_2.54mm:PinSocket_1x01_P2.54mm_Vertical -> Connector_Pin:Pin_D0.7mm_L6.5mm_W1.8mm_FlatFork
- J25: renamed from J27; footprint Connector_PinSocket_2.54mm:PinSocket_1x01_P2.54mm_Vertical -> Connector_Pin:Pin_D0.7mm_L6.5mm_W1.8mm_FlatFork
- J26: renamed from J28; footprint Connector_PinSocket_2.54mm:PinSocket_1x01_P2.54mm_Vertical -> Connector_Pin:Pin_D0.7mm_L6.5mm_W1.8mm_FlatFork
- J3: renamed from J5; footprint Connector_PinSocket_2.54mm:PinSocket_1x01_P2.54mm_Vertical -> Connector_Pin:Pin_D0.7mm_L6.5mm_W1.8mm_FlatFork
- J4: renamed from J6; footprint Connector_PinSocket_2.54mm:PinSocket_1x01_P2.54mm_Vertical -> Connector_Pin:Pin_D0.7mm_L6.5mm_W1.8mm_FlatFork
- J5: renamed from J7; footprint Connector_PinSocket_2.54mm:PinSocket_1x01_P2.54mm_Vertical -> Connector_Pin:Pin_D0.7mm_L6.5mm_W1.8mm_FlatFork
- J6: renamed from J8; footprint Connector_PinSocket_2.54mm:PinSocket_1x01_P2.54mm_Vertical -> Connector_Pin:Pin_D0.7mm_L6.5mm_W1.8mm_FlatFork
- J7: renamed from J9; footprint Connector_PinSocket_2.54mm:PinSocket_1x01_P2.54mm_Vertical -> Connector_Pin:Pin_D0.7mm_L6.5mm_W1.8mm_FlatFork
- J8: renamed from J10; footprint Connector_PinSocket_2.54mm:PinSocket_1x01_P2.54mm_Vertical -> Connector_Pin:Pin_D0.7mm_L6.5mm_W1.8mm_FlatFork
- J9: renamed from J11; footprint Connector_PinSocket_2.54mm:PinSocket_1x01_P2.54mm_Vertical -> Connector_Pin:Pin_D0.7mm_L6.5mm_W1.8mm_FlatFork
- R9: moved to B.Cu
- moved J7 79.6 mm to (124.9, 135.2), turned to 45 degrees
- moved J9 77.6 mm to (118.5, 137.8), turned to 45 degrees
- moved J5 74.3 mm to (123.1, 137.6), turned to 45 degrees
- moved J25 73.3 mm to (122.8, 127.8), turned to 45 degrees
- moved J21 70.0 mm to (124.8, 125.8), turned to 45 degrees
- moved J11 69.6 mm to (113.7, 139.6), turned to 45 degrees
- moved R9 69.0 mm to (107.8, 131.1), turned to -45 degrees
- moved J19 68.8 mm to (126.1, 129.8), turned to 45 degrees
- moved J3 67.5 mm to (120.5, 135.8), turned to 45 degrees
- moved J15 66.4 mm to (110.0, 138.3), turned to 45 degrees
- moved J1 65.5 mm to (123.1, 133.2), turned to 45 degrees
- moved J13 63.4 mm to (115.6, 137.4), turned to 45 degrees
- moved R6 62.3 mm to (118.2, 134.0), turned to -135 degrees
- moved J27 59.5 mm to (104.5, 136.9), turned to -135 degrees
- moved J23 58.8 mm to (127.2, 126.9), turned to 45 degrees
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- renumbered J2 to J27
Routing:
- net Net-(D10-K): track 0.00 -> 175.0 mm, vias 0 -> 5
- net Net-(D1-K): track 0.00 -> 173.9 mm, vias 0 -> 9
- net Net-(D11-K): track 0.00 -> 165.0 mm, vias 0 -> 6
- net Net-(D48-K): track 0.00 -> 153.3 mm, vias 0 -> 7
- net Net-(D12-K): track 0.00 -> 151.4 mm, vias 0 -> 6
- net Net-(D13-K): track 0.00 -> 151.4 mm, vias 0 -> 6
- net Net-(D47-K): track 0.00 -> 134.2 mm, vias 0 -> 6
- net Net-(D46-K): track 0.00 -> 133.1 mm, vias 0 -> 6
- net GND: track 0.00 -> 28.9 mm
- net Net-(D15-K): track 156.7 -> 128.1 mm, vias 6 -> 5
- net +5V: track 0.00 -> 27.6 mm, vias 0 -> 2
- net Net-(U1-PA0): track 10.9 -> 28.3 mm, vias 0 -> 2
- net Net-(D18-K): track 149.2 -> 164.9 mm, vias 7 -> 8
- net Net-(U1-PA6): track 0.00 -> 15.3 mm
- net Net-(D46-A): track 15.6 -> 30.0 mm
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Other:
- board size 103.1 x 218.5 mm -> 89.1 x 194.1 mm

Commit message: selkäsalama mk1 rev 2
Parts:
- J1, J10, J11, J12, J13, J14, J15, J16, J17, J18, J19, J2, J20, J21, J22, J23, J24, J25, J26, J3, J4, J5, J6, J7, J8, J9: footprint Connector_Pin:Pin_D0.7mm_L6.5mm_W1.8mm_FlatFork -> footprinttejä:Pin_D0.8mm_L6.5mm_W1.8mm_FlatFork_zani
- moved J5 31.6 mm to (111.1, 108.3)
- moved J7 31.3 mm to (113.3, 106.2)
- moved J3 27.8 mm to (109.0, 110.5)
- moved R7 27.5 mm to (105.2, 87.1)
- moved J1 27.0 mm to (116.2, 107.1)
- moved R1 26.5 mm to (118.6, 91.4), turned to 45 degrees
- moved J13 26.2 mm to (116.0, 111.1)
- moved J9 25.8 mm to (109.7, 113.5)
- moved J31 25.6 mm to (103.0, 92.4), turned to 45 degrees
- moved J15 25.3 mm to (113.8, 113.3)
- moved R2 24.9 mm to (120.1, 96.5)
- moved J29 24.5 mm to (95.3, 108.5), turned to 45 degrees
- moved J27 24.4 mm to (94.5, 114.6)
- moved J11 24.3 mm to (111.6, 115.4)
- moved J30 24.1 mm to (93.7, 105.6), turned to 45 degrees
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Routing:
- net Net-(D13-K): track 151.4 -> 126.3 mm, vias 6 -> 3
- net Net-(D19-K): track 152.2 -> 129.5 mm, vias 5 -> 2
- net Net-(D10-K): track 175.0 -> 155.7 mm, vias 5 -> 4
- net Net-(D12-K): track 151.4 -> 132.7 mm, vias 6 -> 5
- net Net-(D21-K): track 131.6 -> 115.5 mm, vias 6 -> 4
- net Net-(D18-K): track 164.9 -> 180.7 mm, vias 8 -> 3
- net Net-(D11-K): track 165.0 -> 179.7 mm, vias 6 -> 7
- net Net-(D14-K): track 126.2 -> 114.0 mm, vias 7 -> 3
- net Net-(D1-K): track 173.9 -> 162.9 mm, vias 9 -> 6
- net Net-(D17-K): track 150.0 -> 160.3 mm, vias 3 -> 2
- net Net-(J7-Pin_1): track 12.2 -> 3.74 mm
- net Net-(J5-Pin_1): track 12.3 -> 4.05 mm
- net Net-(D47-K): track 134.2 -> 127.8 mm, vias 6 -> 4
- net Net-(D48-K): track 153.3 -> 147.0 mm, vias 7 -> 3
- net Net-(D20-K): track 124.2 -> 118.6 mm, vias 6 -> 5
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Other:
- board size 89.1 x 194.1 mm -> 97.4 x 216.4 mm
- board text added: ":D"
- board text added: "Röh Röh"
- board text removed: "Zäni"
